Commit message: update

File: udm_urdf/urdf/main.urdf (robot description, URDF)
Before this commit: robot main, 4 links, 3 joints
Links:
- removed link index
- removed link paume
- removed link petit
- removed link pouce
- added link base_link; visual box size=0.08 0.03 0.10
- added link index_phalange_base; visual cylinder length=0.03 radius=0.01
- added link index_phalange_end; visual cylinder length=0.025 radius=0.007
- added link index_phalange_middle; visual cylinder length=0.025 radius=0.009
- added link middle_phalange_base; visual cylinder length=0.03 radius=0.01
- added link middle_phalange_end; visual cylinder length=0.03 radius=0.007
- added link middle_phalange_middle; visual cylinder length=0.03 radius=0.009
- added link pinky_phalange_base; visual cylinder length=0.02 radius=0.005
- added link pinky_phalange_end; visual cylinder length=0.02 radius=0.005
- added link pinky_phalange_middle; visual cylinder length=0.02 radius=0.005
- added link ring_phalange_base; visual cylinder length=0.03 radius=0.01
- added link ring_phalange_end; visual cylinder length=0.025 radius=0.007
- added link ring_phalange_middle; visual cylinder length=0.025 radius=0.009
- added link thumb_phalange_base; visual cylinder length=0.03 radius=0.01
- added link thumb_phalange_end; visual cylinder length=0.02 radius=0.009
Joints:
- removed joint index_to_base
- removed joint petit_to_base
- removed joint pouce_to_base
- added joint base_link_to_index_base: type revolute, parent base_link, child index_phalange_base, origin xyz=0.03 0.0 0.05, axis 1 0 0, limit lower=-1.65 upper=1.57 effort=1000 velocity=0.5
- added joint base_link_to_middle_base: type revolute, parent base_link, child middle_phalange_base, origin xyz=0.008 0.0 0.05, axis 1 0 0, limit lower=-1.65 upper=1.57 effort=1000 velocity=0.5
- added joint base_link_to_pinky_base: type revolute, parent base_link, child pinky_phalange_base, origin xyz=-0.035 0.0 0.05, axis 1 0 0, limit lower=-1.65 upper=1.57 effort=1000 velocity=0.5
- added joint base_link_to_ring_base: type revolute, parent base_link, child ring_phalange_base, origin xyz=-0.015 0.0 0.05, axis 1 0 0, limit lower=-1.65 upper=1.57 effort=1000 velocity=0.5
- added joint index_base_to_middle: type revolute, parent index_phalange_base, child index_phalange_middle, origin xyz=0.0 0.0 0.03, axis 1 0 0, limit lower=-1.65 upper=0 effort=1000 velocity=0.5
- added joint index_middle_to_end: type revolute, parent index_phalange_middle, child index_phalange_end, origin xyz=0.0 0.0 0.025, axis 1 0 0, limit lower=-1.57 upper=0 effort=1000 velocity=0.5
- added joint middle_base_to_middle: type revolute, parent middle_phalange_base, child middle_phalange_middle, origin xyz=0.0 0.0 0.03, axis 1 0 0, limit lower=-1.65 upper=0 effort=1000 velocity=0.5
- added joint middle_middle_to_end: type revolute, parent middle_phalange_middle, child middle_phalange_end, origin xyz=0.0 0.0 0.03, axis 1 0 0, limit lower=-1.57 upper=0 effort=1000 velocity=0.5
- added joint pinky_base_to_middle: type revolute, parent pinky_phalange_base, child pinky_phalange_middle, origin xyz=0.0 0.0 0.02, axis 1 0 0, limit lower=-1.65 upper=0 effort=1000 velocity=0.5
- added joint pinky_middle_to_end: type revolute, parent pinky_phalange_middle, child pinky_phalange_end, origin xyz=0.0 0.0 0.02, axis 1 0 0, limit lower=-1.57 upper=0 effort=1000 velocity=0.5
- added joint ring_base_to_middle: type revolute, parent ring_phalange_base, child ring_phalange_middle, origin xyz=0.0 0.0 0.03, axis 1 0 0, limit lower=-1.65 upper=0 effort=1000 velocity=0.5
- added joint ring_middle_to_end: type revolute, parent ring_phalange_middle, child ring_phalange_end, origin xyz=0.0 0.0 0.025, axis 1 0 0, limit lower=-1.57 upper=0 effort=1000 velocity=0.5
- added joint thumb_base_palm: type revolute, parent base_link, child thumb_phalange_base, origin xyz=0.04 0 -0.025 rpy=0 1.57 0, axis 1 0 0, limit lower=-1.57 upper=0 effort=1000 velocity=0.5
- added joint thumb_end_to_thumb_base: type revolute, parent thumb_phalange_base, child thumb_phalange_end, origin xyz=0 0 0.03 rpy=0 0 0, axis 1 0 0, limit lower=-1.0 upper=0 effort=1000 velocity=0.5
